File: esp12Stack.brd (EAGLE design)
At the start: 31.5 x 30 mm, 23 parts, among them J02 470, J04 470, J05 470, J12 470, J13 470

Commit message: Deep Sleep capability
added a jumper Position to connect GIPO16 and REST to enable wake up from deep sleep.
Parts:
- added J_REST: 10k, eagle-ltspice:R0805
Connections:
- net GPIO16: now also J_REST.1
- net REST: now also J_REST.2
Routing:
- net GPIO16: track 7.27 -> 10.6 mm
- net REST: track 32.8 -> 35.8 mm
- net DOUT2DIN3: track 27.7 -> 29.9 mm
Changed lines of the file:
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@@
 <attribute name="SPICEMODEL" value="NONE" x="7.62" y="16.51" size="1.778" layer="28" rot="MR270" display="off"/>
+</element>
+<element name="J_REST" library="eagle-ltspice" package="R0805" value="10k" x="4.28625" y="16.51" rot="MR90">
+<attribute name="SPICEPREFIX" value="R" x="4.28625" y="16.51" size="1.778" layer="28" rot="MR90" display="off"/>
+<attribute name="SPICEMODEL" value="NONE" x="4.28625" y="16.51" size="1.778" layer="28" rot="MR90" display="off"/>
 </element>
 </elements>
@@
 <contactref element="REST" pad="1"/>
 <wire x1="1.5875" y1="21.59" x2="2.2225" y2="21.59" width="0.254" layer="16"/>
-<wire x1="2.2225" y1="21.59" x2="3.4925" y2="20.32" width="0.254" layer="16"/>
-<wire x1="3.4925" y1="20.32" x2="3.4925" y2="2.3775" width="0.254" layer="16"/>
+<wire x1="2.2225" y1="21.59" x2="4.28625" y2="19.52625" width="0.254" layer="16"/>
 <wire x1="3.4925" y1="2.3775" x2="4.6" y2="1.27" width="0.254" layer="16"/>
+<contactref element="J_REST" pad="2"/>
+<wire x1="4.28625" y1="19.52625" x2="4.28625" y2="17.46" width="0.254" layer="16"/>
+<wire x1="4.28625" y1="17.46" x2="5.24125" y2="17.46" width="0.254" layer="16"/>
+<wire x1="5.24125" y1="17.46" x2="5.55625" y2="17.145" width="0.254" layer="16"/>
+<wire x1="5.55625" y1="17.145" x2="5.55625" y2="14.605" width="0.254" layer="16"/>
+<wire x1="5.55625" y1="14.605" x2="5.08" y2="14.12875" width="0.254" layer="16"/>
+<wire x1="5.08" y1="14.12875" x2="3.81" y2="14.12875" width="0.254" layer="16"/>
+<wire x1="3.81" y1="14.12875" x2="3.4925" y2="13.81125" width="0.254" layer="16"/>
+<wire x1="3.4925" y1="13.81125" x2="3.4925" y2="2.3775" width="0.254" layer="16"/>
 </signal>
 <signal name="ADC">
@@
 <wire x1="2.7432" y1="14.1732" x2="4.92" y2="16.35" width="0.254" layer="1"/>
 <wire x1="4.92" y1="16.35" x2="7.62" y2="16.35" width="0.254" layer="1"/>
+<contactref element="J_REST" pad="1"/>
+<wire x1="1.5875" y1="13.97" x2="2.69625" y2="13.97" width="0.254" layer="16"/>
+<wire x1="2.69625" y1="13.97" x2="4.28625" y2="15.56" width="0.254" layer="16"/>
 </signal>
 <signal name="GPIO14">
@@
 <wire x1="1.905" y1="23.495" x2="2.8575" y2="23.495" width="0.3048" layer="16"/>
 <wire x1="2.8575" y1="23.495" x2="4.1275" y2="22.225" width="0.3048" layer="16"/>
-<wire x1="4.1275" y1="22.225" x2="4.1275" y2="3.81" width="0.3048" layer="16"/>
 <via x="6.0325" y="1.905" extent="1-16" drill="0.6"/>
 <wire x1="4.1275" y1="3.81" x2="6.0325" y2="1.905" width="0.3048" layer="16"/>
 <wire x1="4.2175" y1="1.2075" x2="5.335" y2="1.2075" width="0.3048" layer="1"/>
 <wire x1="5.335" y1="1.2075" x2="6.0325" y2="1.905" width="0.3048" layer="1"/>
+<wire x1="4.1275" y1="22.225" x2="4.1275" y2="20.6375" width="0.254" layer="16"/>
+<wire x1="4.1275" y1="20.6375" x2="4.92125" y2="19.84375" width="0.254" layer="16"/>
+<wire x1="4.92125" y1="19.84375" x2="4.92125" y2="18.89125" width="0.254" layer="16"/>
+<wire x1="4.92125" y1="18.89125" x2="5.3975" y2="18.415" width="0.254" layer="16"/>
+<wire x1="5.3975" y1="18.415" x2="5.3975" y2="17.93875" width="0.254" layer="16"/>
+<wire x1="5.3975" y1="17.93875" x2="6.0325" y2="17.30375" width="0.254" layer="16"/>
+<wire x1="6.0325" y1="17.30375" x2="6.0325" y2="14.2875" width="0.254" layer="16"/>
+<wire x1="6.0325" y1="14.2875" x2="5.23875" y2="13.49375" width="0.254" layer="16"/>
+<wire x1="5.23875" y1="13.49375" x2="4.1275" y2="13.49375" width="0.254" layer="16"/>
+<wire x1="4.1275" y1="13.49375" x2="4.1275" y2="3.81" width="0.254" layer="16"/>
 </signal>
 <signal name="DOUT3DIN4">
