File: esp12StackFTDI_1.sch (EAGLE design)
At the start: 14 parts, among them U1 ESP-WROOM-03

Commit message: FT232 module
FT232 Module now functional as a prototype
Parts:
- removed JP1, JP2, JP3, JP4: (no value), adafruit:PINHD-2X4
- removed U1: ESP-WROOM-03, esp32:ESP-WROOM-03
- added C4: 33n, eagle-ltspice:CC0603
- added IC2: (no value), FTDI:FT232BM
- added J02, J04, J05, J12, J13: 470, eagle-ltspice:RR0603
- added J_REST, R1, R17, R4: 10k, eagle-ltspice:RR0603
- added LED1, LED2, LED3, LED4: WS2812B5050, adafruit:WS2812B5050
- added MDL1: (no value), ESP12E:ESP8266-12EESP8266-ESP12E
- added R12: 470R, eagle-ltspice:RR0603
- added R13, R14: 27R, eagle-ltspice:RR0603
- added R15: 1k4, eagle-ltspice:RR0603
- added R16: 4k7, eagle-ltspice:RR0603
- added SV1, SV2: (no value), con-lstb:MA08-1
- R2, R3, R5: device eagle-ltspice:R -> eagle-ltspice:RR0603
Connections:
- removed net +5V: GND.V_IN, JP2.8, U$2.VCC
- removed net EN: JP1.6, R2.1, REST.1, U1.EN
- removed net GPIO17: JP4.8, U1.IO17
- removed net GPIO18: JP4.6, U1.IO18
- removed net GPIO19: JP4.4, U1.IO19
- removed net GPIO21: JP4.2, U1.IO21
- removed net GPIO22: JP3.8, U1.IO22
- removed net GPIO23: JP3.6, U1.IO23
- removed net GPIO25: JP1.2, U1.IO25
- removed net GPIO27: JP2.7, U1.IO27
- removed net GPIO32: JP2.3, U1.IO32
- removed net GPIO33: JP2.5, U1.IO33
- removed net GPIO34: JP1.5, U1.IO34
- removed net GPIO35: JP1.7, U1.IO35
- new net 3V3OUT1: C4.2, IC2.3V3OUT
- new net 5V: GND.V_IN, IC2.VCC1, IC2.VCC2, LED1.VDD, LED2.VDD, LED3.VDD, LED4.VDD, R12.2, R16.1, SV1.8, U$2.VCC
- new net AVCC1: IC2.AVCC, R12.1
- new net CH_PD: MDL1.CH_PD, R2.1, SV1.3
- new net D+: R14.2, U$2.D+
- new net D-: R13.2, U$2.D-
- new net DIN1: J02.1, J04.1, J05.1, J12.1, J13.1, LED1.DI
- new net DOUT1DIN2: LED1.DO, LED2.DI
- new net DOUT2DIN3: LED2.DO, LED3.DI
- new net DOUT3DIN4: LED3.DO, LED4.DI
- new net RESET1: IC2.RESET, R16.2, R17.1
- new net REST: J_REST.2, MDL1.REST, R1.1, REST.1, SV1.1
- new net RSTOUT1: IC2.RSTOUT, R15.1
- new net USBDM1: IC2.USBDM, R13.1
- new net USBDP1: IC2.USBDP, R14.1, R15.2
- net 3V3: now also IC2.PWRCTL, IC2.VCIO, MDL1.VCC, R1.2, R4.2; no longer U1.3V3
- net ADC: now also MDL1.ADC, SV1.2; no longer JP1.4, U1.SENSOR_VP
- net GND: now also C4.1, IC2.AGND, IC2.GND1, IC2.GND2, LED1.GND, LED2.GND, LED3.GND, LED4.GND, MDL1.GND, R17.2, SV2.8; no longer JP4.7, U1.GND, U1.GND@1, U1.GND@15, U1.GND@38, U1.SENSOR_VN
- net GPIO0: now also MDL1.GPIO0, R4.1, SV2.5; no longer JP4.1, U1.IO0
- net GPIO12: now also J13.2, MDL1.GPIO12, SV1.6; no longer JP2.4, U1.IO12
- net GPIO13: now also J12.2, MDL1.GPIO13, SV1.7; no longer JP2.6, U1.IO13
- net GPIO14: now also MDL1.GPIO14, SV1.5; no longer JP2.2, U1.IO14
- net GPIO15: now also MDL1.GPIO15, SV2.7; no longer JP4.5, U1.IO15
- net GPIO16: now also J_REST.1, MDL1.GPIO16, SV1.4; no longer JP1.8, U1.IO16
- net GPIO2: now also J02.2, MDL1.GPIO2, SV2.6; no longer JP4.3, U1.IO2
- net GPIO4: now also J04.2, MDL1.GPIO4, SV2.4; no longer JP3.7, U1.IO4
- net GPIO5: now also J05.2, MDL1.GPIO5, SV2.3; no longer JP3.5, U1.IO5
- net RXD: now also IC2.TXD, MDL1.RXD, SV2.2; no longer JP3.3, U1.RXD
- net TXD: now also IC2.RXD, MDL1.TXD, SV2.1; no longer JP3.1, U1.TXD
Other:
- note added: "3.3V Power Supply"
- note added: "ESP12 Basics"
- note added: "USB Connector"
- note added: "USB to UART module"
- note added: "WS2812/6824 LEDs (optional)"
